File: Hardware/SinglePhaseEnergyMonitor.kicad_pcb (KiCad board)
At the start: 2 copper layers, 58 x 90 mm, 47 parts, among them J1 Conn_01x03, J2 LED, J3 Conn_01x05, J4 Conn_01x02, M1 ATM90E26_ATM90E26, U1 ESP-07, U2 AT24CS32-STUM, Y1 8.192M

Commit message: improve layout
Parts:
- removed R1: 0R, Resistor_SMD:R_1206_3216Metric
- added J5: Conn_01x01, Connector_Pin:Pin_D0.9mm_L10.0mm_W2.4mm_FlatFork, F.Cu at (126.2, 146.0)
- moved RN1 1.00 mm to (130.0, 146.5)
Connections:
- J1 pad 2: /Neutral_2 -> GND
- PS1 pad 1: /Neutral_2 -> GND
- R3 pad 1: /Neutral_2 -> GND
- R4 pad 2: /Neutral_2 -> GND
Routing:
- net /Neutral_2: track 88.1 -> 0.00 mm
- net GND: track 134.9 -> 203.9 mm
- net +3V3: track 112.2 -> 109.2 mm
- net Net-(RN1-Pad6): track 7.56 -> 8.56 mm
- net CS: track 25.5 -> 26.5 mm
- net Net-(RN1-Pad8): track 7.23 -> 8.23 mm

Commit message: fix pcb
Parts:
- moved J5 1.52 mm to (126.0, 147.5)
Connections:
- J5 pad 1: CS -> Net-(J5-Pad1)
- RN1 pad 6: Net-(RN1-Pad6) -> Net-(J5-Pad1)
- U1 pad 12: Net-(RN1-Pad6) -> Net-(J5-Pad1)
Routing:
- net Net-(J5-Pad1): track 0.00 -> 9.67 mm
- net Net-(RN1-Pad6): track 8.56 -> 0.00 mm
