File: Hardware/SinglePhaseEnergyMonitor.sch (KiCad schematic (older format))
At the start: 47 parts, among them J1 Conn_01x03, J2 LED, J3 Conn_01x05, J4 Conn_01x02, M1 ATM90E26_ATM90E26, U1 ESP-07, U2 AT24CS32-STUM, Y1 8.192M

Commit message: improve layout
Parts:
- removed R1: 0R, Resistor_SMD:R_1206_3216Metric, symbol Device:R
- added J5: Conn_01x01, Connector_Pin:Pin_D0.9mm_L10.0mm_W2.4mm_FlatFork, symbol Connector_Generic:Conn_01x01
Connections:
- net Neutral_2 is gone; now on net GND: J1.2 (Pin_2), PS1.1 (AC/N), R3.1, R4.2
- net CS: now also J5.1 (Pin_1)
Changed lines of the file:
@@
 	3950 5050 4100 5050
-$Comp
-L Device:R R1
-U 1 1 5C21BB38
-P 2800 2650
-F 0 "R1" V 3000 2650 50  0000 C CNN
-F 1 "0R" V 2900 2650 50  0000 C CNN
-F 2 "Resistor_SMD:R_1206_3216Metric" V 2730 2650 50  0001 C CNN
-F 3 "~" H 2800 2650 50  0001 C CNN
-	1    2800 2650
-	-1   0    0    1
-$EndComp
 $Comp
 L power:GND #PWR0119
@@
 	1    0    0    -1
 $EndComp
-Wire Wire Line
-	2800 2850 2800 2800
 $Comp
 L RF_Module:ESP-07 U1
@@
 Wire Wire Line
 	2450 2450 2800 2450
-Wire Wire Line
-	2800 2450 2800 2500
 Connection ~ 2450 2450
 Wire Wire Line
@@
 Wire Wire Line
 	8300 3550 8300 4800
-Text GLabel 8400 3750 2    50   Input ~ 0
+Text GLabel 8650 3650 2    50   Input ~ 0
 CS
-Wire Wire Line
-	8400 3750 8200 3750
 Connection ~ 8200 3750
 Wire Wire Line
@@
 	0    -1   -1   0
 $EndComp
+Wire Wire Line
+	2800 2450 2800 2850
+$Comp
+L Connector_Generic:Conn_01x01 J5
+U 1 1 5C239DDC
+P 8850 3800
+F 0 "J5" H 8930 3842 50  0000 L CNN
+F 1 "Conn_01x01" H 8930 3751 50  0000 L CNN
+F 2 "Connector_Pin:Pin_D0.9mm_L10.0mm_W2.4mm_FlatFork" H 8850 3800 50  0001 C CNN
+F 3 "~" H 8850 3800 50  0001 C CNN
+	1    8850 3800
+	1    0    0    -1
+$EndComp
+Wire Wire Line
+	8650 3650 8550 3650
+Wire Wire Line
+	8550 3650 8550 3750
+Wire Wire Line
+	8550 3800 8650 3800
+Wire Wire Line
+	8200 3750 8550 3750
+Connection ~ 8550 3750
+Wire Wire Line
+	8550 3750 8550 3800
 $EndSCHEMATC

Commit message: fix pcb
Connections:
- net CS: no longer J5.1 (Pin_1)
- net at RN1.6 (R3.2), U1.12 (GPIO0): now also J5.1 (Pin_1)
Changed lines of the file:
@@
 	8200 3750 8200 4800
 Wire Wire Line
-	8300 3550 8300 4800
+	8300 3550 8300 3800
 Text GLabel 8650 3650 2    50   Input ~ 0
 CS
@@
 	8550 3650 8550 3750
 Wire Wire Line
-	8550 3800 8650 3800
+	8200 3750 8550 3750
 Wire Wire Line
-	8200 3750 8550 3750
-Connection ~ 8550 3750
+	8300 3800 8650 3800
+Connection ~ 8300 3800
 Wire Wire Line
-	8550 3750 8550 3800
+	8300 3800 8300 4800
 $EndSCHEMATC
